File: attachment_processor_4/attachment_processor_4.kicad_sch (KiCad schematic)
At the start: 143 parts, among them U1 TMS4256, U10 TMS4256, U100 74ALS576, U101 74ALS842, U102 74ALS841, U103 MC1488, U104 WD1943-PD, U105 TIBPAL16R8, U106 PAL16P8, U107 74ALS576, U108 74ALS841, U109 MC1488, U11 TMS4256, U110 74ALS244, U111 P8274, U112 TIBPAL16R8, U113 TIBPAL16R6, U114 74ALS240, U115 74ALS576, U116 74ALS240, U117 MC1488, U118 74ALS257, U119 PAL16L8, U12 TMS4256, U120 74ALS832, U121 TIBPAL16L8, U122 PAL20L8, U124 MC1489, U125 74ALS161, U126 PAL16R4, U127 TIBPAL16R4, U128 74ALS161, U129 74LS125, U13 TMS4256, U130 74ALS874, U131 74AS576, U132 74ALS257, U133 P8274, U134 PAL16R6, U135 74AS74, U136 PAL16L8, U137 74LS125, U138 74AS1004, U139 74AS161, U14 TMS4256, U140 74AS161, U15 TMS4256, U16 TMS4256, U17 TMS4256, U18 TMS4256, U19 MB81C4256, U2 TMS4256, U20 MB81C4256, U21 MB81C4256, U22 MB81C4256, U23 74F657, U24 74F657, U25 74F657, U26 74F657, U27 TMS4256, U28 TMS4256, U29 TMS4256, U3 TMS4256, U30 TMS4256, U31 TMS4256, U32 TMS4256, U33 TMS4256, U34 TMS4256, U35 TMS4256, U36 TMS4256, U37 TMS4256, U38 TMS4256, U39 TMS4256, U4 TMS4256, U40 TMS4256, U41 TMS4256, U42 TMS4256, U43 TMS4256, U44 TMS4256, U45 MB81C4256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

Commit message: AP: Trace data bus
Connections:
- net ##64: now reaches U11.14 (Q)
- net ##64: now also U11.2 (D), U19.1 (DQ1), U2.14 (Q), U2.2 (D), U24.14 (B7), U25.14 (B7), U45.1 (DQ1)
- net ##70: now reaches U30.14 (Q)
- net ##70: now also U21.18 (DQ3), U26.16 (B5), U30.2 (D), U39.14 (Q), U39.2 (D), U47.18 (DQ3)
- net ##57: now reaches U9.14 (Q)
- net ##57: now also U18.14 (Q), U18.2 (D), U20.19 (DQ4), U24.23 (B0), U25.23 (B0), U46.19 (DQ4), U9.2 (D)
- net ##68: now reaches U48.1 (DQ1)
- net ##68: now also U22.1 (DQ1), U26.20 (B3), U32.14 (Q), U32.2 (D), U41.14 (Q), U41.2 (D)
- net ##66: now reaches U48.18 (DQ3)
- net ##66: now also U22.18 (DQ3), U26.22 (B1), U34.14 (Q), U34.2 (D), U43.14 (Q), U43.2 (D)
- net ##65: now reaches U48.19 (DQ4)
- net ##65: now also U22.19 (DQ4), U26.23 (B0), U35.14 (Q), U35.2 (D), U44.14 (Q), U44.2 (D)
- net ##67: now reaches U48.2 (DQ2)
- net ##67: now also U22.2 (DQ2), U26.21 (B2), U33.14 (Q), U33.2 (D), U42.14 (Q), U42.2 (D)
- net ##8: now reaches U111.12 (DB7)
- net ##8: now also U107.12 (8~{Q}), U114.12 (O3a), U115.12 (8~{Q}), U133.12 (DB7), U53.18 (D_{7}), U54.19 (D7), U69.18 (D7), U71.14 (O8), U72.11 (B8), U74.62 (D7), U89.18 (D7), U90.12 (DB7)
- net ##7: now reaches U111.13 (DB6)
- net ##7: now also U107.13 (7~{Q}), U114.14 (O2a), U115.13 (7~{Q}), U133.13 (DB6), U53.19 (D_{6}), U54.18 (D6), U69.17 (D6), U71.13 (O7), U72.12 (B7), U74.63 (D6), U89.17 (D6), U90.13 (DB6)
- net ##6: now reaches U111.14 (DB5)
- net ##6: now also U107.14 (6~{Q}), U114.16 (O1a), U115.14 (6~{Q}), U133.14 (DB5), U53.20 (D_{5}), U54.17 (D5), U69.14 (D5), U71.12 (O6), U72.13 (B6), U74.64 (D5), U89.14 (D5), U90.14 (DB5)
- net ##5: now reaches U111.15 (DB4)
- net ##5: now also U107.15 (5~{Q}), U114.18 (O0a), U115.15 (5~{Q}), U133.15 (DB4), U53.21 (D_{4}), U54.16 (D4), U69.13 (D4), U71.11 (O5), U72.14 (B5), U74.1 (D4), U89.13 (D4), U90.15 (DB4)
- net ##4: now reaches U111.16 (DB3)
- net ##4: now also U107.16 (4~{Q}), U114.3 (O3b), U115.16 (4~{Q}), U133.16 (DB3), U53.22 (D_{3}), U54.15 (D3), U69.8 (D3), U71.9 (O4), U72.15 (B4), U74.2 (D3), U89.8 (D3), U90.16 (DB3)
- net ##3: now reaches U111.17 (DB2)
- net ##3: now also U107.17 (3~{Q}), U114.5 (O2b), U115.17 (3~{Q}), U133.17 (DB2), U53.23 (D_{2}), U54.13 (D2), U69.7 (D2), U71.8 (O3), U72.16 (B3), U74.3 (D2), U89.7 (D2), U90.17 (DB2)
- net ##2: now reaches U111.18 (DB1)
- net ##2: now also U106.12 (O8), U107.18 (2~{Q}), U114.7 (O1b), U115.18 (2~{Q}), U133.18 (DB1), U53.24 (D_{1}), U54.12 (D1), U69.4 (D1), U71.7 (O2), U72.17 (B2), U74.4 (D1), U89.4 (D1), U90.18 (DB1)
- net ##1: now reaches U111.19 (DB0)
- net ##1: now also U106.15 (IO5), U107.19 (1~{Q}), U114.9 (O0b), U115.19 (1~{Q}), U133.19 (DB0), U53.25 (D_{0}), U54.11 (D0), U69.3 (D0), U71.6 (O1), U72.18 (B1), U74.5 (D0), U89.3 (D0), U90.19 (DB0), U97.23 (O0)
- net ##32: now reaches U62.1 (DQ1)
- net ##32: now also U80.14 (B7)
- net ##30: now reaches U62.18 (DQ3)
- net ##30: now also U80.16 (B5)
- net ##29: now reaches U62.19 (DQ4)
- net ##29: now also U80.17 (B4)
- net ##31: now reaches U62.2 (DQ2)
- net ##31: now also U80.15 (B6)
- net ##9: now reaches U55.11 (D0)
- net ##9: now also U100.19 (1~{Q}), U131.19 (1~{Q}), U49.18 (B1), U74.61 (D8), U92.3 (D0)
- net ##10: now reaches U55.12 (D1)
- net ##10: now also U100.18 (2~{Q}), U131.18 (2~{Q}), U49.17 (B2), U74.60 (D9), U92.4 (D1)
- net ##11: now reaches U55.13 (D2)
- net ##11: now also U100.17 (3~{Q}), U131.17 (3~{Q}), U49.16 (B3), U74.59 (D10), U92.7 (D2)
- net ##12: now reaches U55.15 (D3)
- net ##12: now also U100.16 (4~{Q}), U131.16 (4~{Q}), U49.15 (B4), U74.58 (D11), U92.8 (D3)
- net ##13: now reaches U55.16 (D4)
- net ##13: now also U100.15 (5~{Q}), U131.15 (5~{Q}), U49.14 (B5), U74.57 (D12), U92.13 (D4)
- net ##14: now reaches U55.17 (D5)
- net ##14: now also U100.14 (6~{Q}), U131.14 (6~{Q}), U49.13 (B6), U74.56 (D13), U92.14 (D5)
- net ##15: now reaches U55.18 (D6)
- net ##15: now also U100.13 (7~{Q}), U131.13 (7~{Q}), U49.12 (B7), U74.55 (D14), U92.17 (D6)
- net ##16: now reaches U55.19 (D7)
- net ##16: now also U100.12 (8~{Q}), U131.12 (8~{Q}), U49.11 (B8), U74.54 (D15), U92.18 (D7)
- net ##104: now reaches U67.14 (Q)
- net ##104: now also U26.13 (PARITY), U27.14 (Q), U27.2 (D), U36.14 (Q), U36.2 (D), U65.14 (Q), U65.2 (D), U67.2 (D)
- net ##103: now reaches U1.14 (Q)
- net ##103: now also U1.2 (D), U10.14 (Q), U10.2 (D), U24.13 (PARITY), U25.13 (PARITY), U64.14 (Q), U64.2 (D), U66.14 (Q), U66.2 (D)
- net ##62: now reaches U45.18 (DQ3)
- net ##62: now also U13.14 (Q), U13.2 (D), U19.18 (DQ3), U24.16 (B5), U25.16 (B5), U4.14 (Q), U4.2 (D)
- net ##61: now reaches U45.19 (DQ4)
- net ##61: now also U14.14 (Q), U14.2 (D), U19.19 (DQ4), U24.17 (B4), U25.17 (B4), U5.14 (Q), U5.2 (D)
- net ##63: now reaches U45.2 (DQ2)
- net ##63: now also U12.14 (Q), U12.2 (D), U19.2 (DQ2), U24.15 (B6), U25.15 (B6), U3.14 (Q), U3.2 (D)
- net ##69: now reaches U31.14 (Q)
- net ##69: now also U21.19 (DQ4), U26.17 (B4), U31.2 (D), U40.14 (Q), U40.2 (D), U47.19 (DQ4)
- net ##41: now reaches U49.2 (A1)
- net ##41: now also U23.2 (A0), U51.2 (A1), U52.2 (A1)
- net ##42: now reaches U49.3 (A2)
- net ##42: now also U23.3 (A1), U51.3 (A2), U52.3 (A2)
- net ##43: now reaches U49.4 (A3)
- net ##43: now also U23.4 (A2), U51.4 (A3), U52.4 (A3)
- net ##44: now reaches U49.5 (A4)
- net ##44: now also U23.5 (A3), U51.5 (A4), U52.5 (A4)
- net ##45: now reaches U49.6 (A5)
- net ##45: now also U23.6 (A4), U51.6 (A5), U52.6 (A5)
- net ##46: now reaches U49.7 (A6)
- net ##46: now also U23.8 (A5), U51.7 (A6), U52.7 (A6)
- net ##47: now reaches U49.8 (A7)
- net ##47: now also U23.9 (A6), U51.8 (A7), U52.8 (A7)
- net ##48: now reaches U49.9 (A8)
- net ##48: now also U23.10 (A7), U51.9 (A8), U52.9 (A8)
- net ##56: now reaches U70.11 (B8)
- net ##56: now also U24.10 (A7), U26.10 (A7), U52.11 (B8)
- net ##55: now reaches U70.12 (B7)
- net ##55: now also U24.9 (A6), U26.9 (A6), U52.12 (B7)
- net ##54: now reaches U70.13 (B6)
- net ##54: now also U24.8 (A5), U26.8 (A5), U52.13 (B6)
- net ##53: now reaches U70.14 (B5)
- net ##53: now also U24.6 (A4), U26.6 (A4), U52.14 (B5)
- net ##52: now reaches U70.15 (B4)
- net ##52: now also U24.5 (A3), U26.5 (A3), U52.15 (B4)
- net ##51: now reaches U70.16 (B3)
- net ##51: now also U24.4 (A2), U26.4 (A2), U52.16 (B3)
- net ##50: now reaches U70.17 (B2)
- net ##50: now also U24.3 (A1), U26.3 (A1), U52.17 (B2)
- net ##49: now reaches U70.18 (B1)
- net ##49: now also U24.2 (A0), U26.2 (A0), U52.18 (B1)
- net ##17: now reaches U70.2 (A1)
- net ##17: now also U72.2 (A1), U80.2 (A0)
- net ##18: now reaches U70.3 (A2)
- net ##18: now also U72.3 (A2), U80.3 (A1)
- net ##19: now reaches U70.4 (A3)
- net ##19: now also U72.4 (A3), U80.4 (A2)
- net ##20: now reaches U70.5 (A4)
- net ##20: now also U72.5 (A4), U80.5 (A3)
- net ##21: now reaches U70.6 (A5)
- net ##21: now also U72.6 (A5), U80.6 (A4)
- net ##22: now reaches U70.7 (A6)
- net ##22: now also U72.7 (A6), U80.8 (A5)
- net ##23: now reaches U70.8 (A7)
- net ##23: now also U72.8 (A7), U80.9 (A6)
- net ##24: now reaches U70.9 (A8)
- net ##24: now also U72.9 (A8), U80.10 (A7)
- net ##72: now reaches U28.14 (Q)
- net ##72: now also U21.1 (DQ1), U26.14 (B7), U28.2 (D), U37.14 (Q), U37.2 (D), U47.1 (DQ1)
- net ##58: now reaches U8.14 (Q)
- net ##58: now also U17.14 (Q), U17.2 (D), U20.18 (DQ3), U24.22 (B1), U25.22 (B1), U46.18 (DQ3), U8.2 (D)
- net ##101: now reaches U61.14 (Q)
- net ##101: now also U61.2 (D), U80.13 (PARITY)
- net ##59: now reaches U7.14 (Q)
- net ##59: now also U16.14 (Q), U16.2 (D), U20.2 (DQ2), U24.21 (B2), U25.21 (B2), U46.2 (DQ2), U7.2 (D)
- net ##28: now reaches U63.1 (DQ1)
- net ##28: now also U80.20 (B3)
- net ##26: now reaches U63.18 (DQ3)
- net ##26: now also U80.22 (B1)
- net ##25: now reaches U63.19 (DQ4)
- net ##25: now also U80.23 (B0)
- net ##27: now reaches U63.2 (DQ2)
- net ##27: now also U80.21 (B2)
- net ##71: now reaches U47.2 (DQ2)
- net ##71: now also U21.2 (DQ2), U26.15 (B6), U29.14 (Q), U29.2 (D), U38.14 (Q), U38.2 (D)
- net ##40: now reaches U59.1 (DQ1)
- net ##40: now also U23.14 (B7)
- net ##38: now reaches U59.18 (DQ3)
- net ##38: now also U23.16 (B5)
- net ##37: now reaches U59.19 (DQ4)
- net ##37: now also U23.17 (B4)
- net ##39: now reaches U59.2 (DQ2)
- net ##39: now also U23.15 (B6)
- net ##102: now reaches U23.13 (PARITY)
- net ##102: now also U58.14 (Q), U58.2 (D)
- net ##36: now reaches U23.20 (B3)
- net ##36: now also U60.1 (DQ1)
- net ##35: now reaches U23.21 (B2)
- net ##35: now also U60.2 (DQ2)
- net ##34: now reaches U23.22 (B1)
- net ##34: now also U60.18 (DQ3)
- net ##33: now reaches U23.23 (B0)
- net ##33: now also U60.19 (DQ4)
- net ##60: now reaches U15.14 (Q)
- net ##60: now also U15.2 (D), U20.1 (DQ1), U24.20 (B3), U25.20 (B3), U46.1 (DQ1), U6.14 (Q), U6.2 (D)
- net ##80: now reaches U25.10 (A7)
- net ##80: now also U51.11 (B8)
- net ##73: now reaches U25.2 (A0)
- net ##73: now also U51.18 (B1)
- net ##74: now reaches U25.3 (A1)
- net ##74: now also U51.17 (B2)
- net ##75: now reaches U25.4 (A2)
- net ##75: now also U51.16 (B3)
- net ##76: now reaches U25.5 (A3)
- net ##76: now also U51.15 (B4)
- net ##77: now reaches U25.6 (A4)
- net ##77: now also U51.14 (B5)
- net ##78: now reaches U25.8 (A5)
- net ##78: now also U51.13 (B6)
- net ##79: now reaches U25.9 (A6)
- net ##79: now also U51.12 (B7)

Commit message: AP: Trace address bus
Parts:
- added RN1: R_Network09_US, Resistor_THT:R_Array_SIP10, symbol Device:R_Network09_US
Connections:
- net ##258: now reaches U83.10 (I10)
- net ##258: now also U74.47 (A19), U84.5 (4D)
- net ##257: now reaches U83.11 (I11)
- net ##257: now also U74.46 (A18), U84.4 (3D), U86.10 (9D), U86.11 (10D)
- net ##256: now reaches U83.13 (I12)
- net ##256: now also U74.45 (A17), U84.3 (2D), U86.9 (8D)
- net ##255: now reaches U83.14 (O10)
- net ##255: now also U74.44 (A16), U84.2 (1D), U86.8 (7D), W1.6 (Pin_6)
- net ##262: now reaches U83.6 (I6)
- net ##262: now also U74.52 (A23), U84.9 (8D)
- net ##261: now reaches U83.7 (I7)
- net ##261: now also U74.51 (A22), U84.8 (7D)
- net ##260: now reaches U83.8 (I8)
- net ##260: now also U74.50 (A21), U84.7 (6D)
- net ##259: now reaches U83.9 (I9)
- net ##259: now also U74.48 (A20), U84.6 (5D)
- net ##209: now reaches U11.1 (A8)
- net ##209: now also U1.1 (A8), U10.1 (A8), U102.15 (9Q), U108.15 (9Q), U12.1 (A8), U13.1 (A8), U14.1 (A8), U15.1 (A8), U16.1 (A8), U17.1 (A8), U18.1 (A8), U19.15 (A8), U2.1 (A8), U20.15 (A8), U21.15 (A8), U22.15 (A8), U27.1 (A8), U28.1 (A8), U29.1 (A8), U3.1 (A8), U30.1 (A8), U31.1 (A8), U32.1 (A8), U33.1 (A8), U34.1 (A8), U35.1 (A8), U36.1 (A8), U37.1 (A8), U38.1 (A8), U39.1 (A8), U4.1 (A8), U40.1 (A8), U41.1 (A8), U42.1 (A8), U43.1 (A8), U44.1 (A8), U45.15 (A8), U46.15 (A8), U47.15 (A8), U48.15 (A8), U5.1 (A8), U6.1 (A8), U64.1 (A8), U65.1 (A8), U66.1 (A8), U67.1 (A8), U7.1 (A8), U8.1 (A8), U9.1 (A8)
- net ##206: now reaches U11.10 (A5)
- net ##206: now also U1.10 (A5), U10.10 (A5), U102.18 (6Q), U108.18 (6Q), U12.10 (A5), U13.10 (A5), U14.10 (A5), U15.10 (A5), U16.10 (A5), U17.10 (A5), U18.10 (A5), U19.12 (A5), U2.10 (A5), U20.12 (A5), U21.12 (A5), U22.12 (A5), U27.10 (A5), U28.10 (A5), U29.10 (A5), U3.10 (A5), U30.10 (A5), U31.10 (A5), U32.10 (A5), U33.10 (A5), U34.10 (A5), U35.10 (A5), U36.10 (A5), U37.10 (A5), U38.10 (A5), U39.10 (A5), U4.10 (A5), U40.10 (A5), U41.10 (A5), U42.10 (A5), U43.10 (A5), U44.10 (A5), U45.12 (A5), U46.12 (A5), U47.12 (A5), U48.12 (A5), U5.10 (A5), U6.10 (A5), U64.10 (A5), U65.10 (A5), U66.10 (A5), U67.10 (A5), U7.10 (A5), U8.10 (A5), U9.10 (A5)
- net ##205: now reaches U11.11 (A4)
- net ##205: now also U1.11 (A4), U10.11 (A4), U102.19 (5Q), U108.19 (5Q), U12.11 (A4), U13.11 (A4), U14.11 (A4), U15.11 (A4), U16.11 (A4), U17.11 (A4), U18.11 (A4), U19.11 (A4), U2.11 (A4), U20.11 (A4), U21.11 (A4), U22.11 (A4), U27.11 (A4), U28.11 (A4), U29.11 (A4), U3.11 (A4), U30.11 (A4), U31.11 (A4), U32.11 (A4), U33.11 (A4), U34.11 (A4), U35.11 (A4), U36.11 (A4), U37.11 (A4), U38.11 (A4), U39.11 (A4), U4.11 (A4), U40.11 (A4), U41.11 (A4), U42.11 (A4), U43.11 (A4), U44.11 (A4), U45.11 (A4), U46.11 (A4), U47.11 (A4), U48.11 (A4), U5.11 (A4), U6.11 (A4), U64.11 (A4), U65.11 (A4), U66.11 (A4), U67.11 (A4), U7.11 (A4), U8.11 (A4), U9.11 (A4)
- net ##204: now reaches U11.12 (A3)
- net ##204: now also U1.12 (A3), U10.12 (A3), U102.20 (4Q), U108.20 (4Q), U12.12 (A3), U13.12 (A3), U14.12 (A3), U15.12 (A3), U16.12 (A3), U17.12 (A3), U18.12 (A3), U19.9 (A3), U2.12 (A3), U20.9 (A3), U21.9 (A3), U22.9 (A3), U27.12 (A3), U28.12 (A3), U29.12 (A3), U3.12 (A3), U30.12 (A3), U31.12 (A3), U32.12 (A3), U33.12 (A3), U34.12 (A3), U35.12 (A3), U36.12 (A3), U37.12 (A3), U38.12 (A3), U39.12 (A3), U4.12 (A3), U40.12 (A3), U41.12 (A3), U42.12 (A3), U43.12 (A3), U44.12 (A3), U45.9 (A3), U46.9 (A3), U47.9 (A3), U48.9 (A3), U5.12 (A3), U6.12 (A3), U64.12 (A3), U65.12 (A3), U66.12 (A3), U67.12 (A3), U7.12 (A3), U8.12 (A3), U9.12 (A3)
- net ##207: now reaches U11.13 (A6)
- net ##207: now also U1.13 (A6), U10.13 (A6), U102.17 (7Q), U108.17 (7Q), U12.13 (A6), U13.13 (A6), U14.13 (A6), U15.13 (A6), U16.13 (A6), U17.13 (A6), U18.13 (A6), U19.13 (A6), U2.13 (A6), U20.13 (A6), U21.13 (A6), U22.13 (A6), U27.13 (A6), U28.13 (A6), U29.13 (A6), U3.13 (A6), U30.13 (A6), U31.13 (A6), U32.13 (A6), U33.13 (A6), U34.13 (A6), U35.13 (A6), U36.13 (A6), U37.13 (A6), U38.13 (A6), U39.13 (A6), U4.13 (A6), U40.13 (A6), U41.13 (A6), U42.13 (A6), U43.13 (A6), U44.13 (A6), U45.13 (A6), U46.13 (A6), U47.13 (A6), U48.13 (A6), U5.13 (A6), U6.13 (A6), U64.13 (A6), U65.13 (A6), U66.13 (A6), U67.13 (A6), U7.13 (A6), U8.13 (A6), U9.13 (A6)
- net ##108: now reaches U11.15 (~{CAS})
- net ##108: now also U10.15 (~{CAS}), U12.15 (~{CAS}), U120.6, U13.15 (~{CAS}), U14.15 (~{CAS}), U15.15 (~{CAS}), U16.15 (~{CAS}), U17.15 (~{CAS}), U18.15 (~{CAS}), U36.15 (~{CAS}), U37.15 (~{CAS}), U38.15 (~{CAS}), U39.15 (~{CAS}), U40.15 (~{CAS}), U41.15 (~{CAS}), U42.15 (~{CAS}), U43.15 (~{CAS}), U44.15 (~{CAS})
- net ##201: now reaches U11.5 (A0)
- net ##201: now also U1.5 (A0), U10.5 (A0), U102.23 (1Q), U108.23 (1Q), U12.5 (A0), U13.5 (A0), U14.5 (A0), U15.5 (A0), U16.5 (A0), U17.5 (A0), U18.5 (A0), U19.6 (A0), U2.5 (A0), U20.6 (A0), U21.6 (A0), U22.6 (A0), U27.5 (A0), U28.5 (A0), U29.5 (A0), U3.5 (A0), U30.5 (A0), U31.5 (A0), U32.5 (A0), U33.5 (A0), U34.5 (A0), U35.5 (A0), U36.5 (A0), U37.5 (A0), U38.5 (A0), U39.5 (A0), U4.5 (A0), U40.5 (A0), U41.5 (A0), U42.5 (A0), U43.5 (A0), U44.5 (A0), U45.6 (A0), U46.6 (A0), U47.6 (A0), U48.6 (A0), U5.5 (A0), U6.5 (A0), U64.5 (A0), U65.5 (A0), U66.5 (A0), U67.5 (A0), U7.5 (A0), U8.5 (A0), U9.5 (A0)
- net ##203: now reaches U11.6 (A2)
- net ##203: now also U1.6 (A2), U10.6 (A2), U102.21 (3Q), U108.21 (3Q), U12.6 (A2), U13.6 (A2), U14.6 (A2), U15.6 (A2), U16.6 (A2), U17.6 (A2), U18.6 (A2), U19.8 (A2), U2.6 (A2), U20.8 (A2), U21.8 (A2), U22.8 (A2), U27.6 (A2), U28.6 (A2), U29.6 (A2), U3.6 (A2), U30.6 (A2), U31.6 (A2), U32.6 (A2), U33.6 (A2), U34.6 (A2), U35.6 (A2), U36.6 (A2), U37.6 (A2), U38.6 (A2), U39.6 (A2), U4.6 (A2), U40.6 (A2), U41.6 (A2), U42.6 (A2), U43.6 (A2), U44.6 (A2), U45.8 (A2), U46.8 (A2), U47.8 (A2), U48.8 (A2), U5.6 (A2), U6.6 (A2), U64.6 (A2), U65.6 (A2), U66.6 (A2), U67.6 (A2), U7.6 (A2), U8.6 (A2), U9.6 (A2)
- net ##202: now reaches U11.7 (A1)
- net ##202: now also U1.7 (A1), U10.7 (A1), U102.22 (2Q), U108.22 (2Q), U12.7 (A1), U13.7 (A1), U14.7 (A1), U15.7 (A1), U16.7 (A1), U17.7 (A1), U18.7 (A1), U19.7 (A1), U2.7 (A1), U20.7 (A1), U21.7 (A1), U22.7 (A1), U27.7 (A1), U28.7 (A1), U29.7 (A1), U3.7 (A1), U30.7 (A1), U31.7 (A1), U32.7 (A1), U33.7 (A1), U34.7 (A1), U35.7 (A1), U36.7 (A1), U37.7 (A1), U38.7 (A1), U39.7 (A1), U4.7 (A1), U40.7 (A1), U41.7 (A1), U42.7 (A1), U43.7 (A1), U44.7 (A1), U45.7 (A1), U46.7 (A1), U47.7 (A1), U48.7 (A1), U5.7 (A1), U6.7 (A1), U64.7 (A1), U65.7 (A1), U66.7 (A1), U67.7 (A1), U7.7 (A1), U8.7 (A1), U9.7 (A1)
- net ##208: now reaches U11.9 (A7)
- net ##208: now also U1.9 (A7), U10.9 (A7), U102.16 (8Q), U108.16 (8Q), U12.9 (A7), U13.9 (A7), U14.9 (A7), U15.9 (A7), U16.9 (A7), U17.9 (A7), U18.9 (A7), U19.14 (A7), U2.9 (A7), U20.14 (A7), U21.14 (A7), U22.14 (A7), U27.9 (A7), U28.9 (A7), U29.9 (A7), U3.9 (A7), U30.9 (A7), U31.9 (A7), U32.9 (A7), U33.9 (A7), U34.9 (A7), U35.9 (A7), U36.9 (A7), U37.9 (A7), U38.9 (A7), U39.9 (A7), U4.9 (A7), U40.9 (A7), U41.9 (A7), U42.9 (A7), U43.9 (A7), U44.9 (A7), U45.14 (A7), U46.14 (A7), U47.14 (A7), U48.14 (A7), U5.9 (A7), U6.9 (A7), U64.9 (A7), U65.9 (A7), U66.9 (A7), U67.9 (A7), U7.9 (A7), U8.9 (A7), U9.9 (A7)
- net ##109: now reaches U30.15 (~{CAS})
- net ##109: now also U1.15 (~{CAS}), U2.15 (~{CAS}), U27.15 (~{CAS}), U28.15 (~{CAS}), U29.15 (~{CAS}), U3.15 (~{CAS}), U31.15 (~{CAS}), U32.15 (~{CAS}), U33.15 (~{CAS}), U34.15 (~{CAS}), U35.15 (~{CAS}), U4.15 (~{CAS}), U5.15 (~{CAS}), U6.15 (~{CAS}), U7.15 (~{CAS}), U75.3, U8.15 (~{CAS}), U9.15 (~{CAS})
- net ##107: now reaches U48.17 (~{CAS})
- net ##107: now also U45.17 (~{CAS}), U46.17 (~{CAS}), U47.17 (~{CAS}), U64.15 (~{CAS}), U65.15 (~{CAS}), U75.14
- net ##240: now reaches U111.24 (A1)
- net ##240: now also U133.24 (A1), U134.8 (I8), U138.9, U50.6 (A0), U54.10 (A0), U55.10 (A0), U74.29 (A1), U79.2 (1D), U81.3 (2D), U90.24 (A1), U94.1 (A0)
- net ##241: now reaches U111.25 (A0)
- net ##241: now also U133.25 (A0), U134.7 (I7), U138.11, U50.7 (A1), U54.9 (A1), U55.9 (A1), U74.30 (A2), U79.3 (2D), U81.4 (3D), U90.25 (A0), U94.2 (A1)
- net ##214: now reaches U62.11 (A4)
- net ##214: now also U101.19 (5Q), U58.11 (A4), U59.11 (A4), U60.11 (A4), U61.11 (A4), U63.11 (A4), U79.19 (5Q), U86.19 (5Q), U87.19 (5Q)
- net ##215: now reaches U62.12 (A5)
- net ##215: now also U101.18 (6Q), U58.10 (A5), U59.12 (A5), U60.12 (A5), U61.10 (A5), U63.12 (A5), U79.18 (6Q), U86.18 (6Q), U87.18 (6Q)
- net ##216: now reaches U62.13 (A6)
- net ##216: now also U101.17 (7Q), U58.13 (A6), U59.13 (A6), U60.13 (A6), U61.13 (A6), U63.13 (A6), U79.17 (7Q), U86.17 (7Q), U87.17 (7Q)
- net ##217: now reaches U62.14 (A7)
- net ##217: now also U101.16 (8Q), U58.9 (A7), U59.14 (A7), U60.14 (A7), U61.9 (A7), U63.14 (A7), U79.16 (8Q), U86.16 (8Q), U87.16 (8Q)
- net ##218: now reaches U62.15 (A8)
- net ##218: now also U101.15 (9Q), U58.1 (A8), U59.15 (A8), U60.15 (A8), U61.1 (A8), U63.15 (A8), U79.15 (9Q), U86.15 (9Q), U87.15 (9Q)
- net ##105: now reaches U62.17 (~{CAS})
- net ##105: now also U110.14 (O2a), U58.15 (~{CAS}), U59.17 (~{CAS}), U60.17 (~{CAS}), U61.15 (~{CAS}), U63.17 (~{CAS})
- net ##210: now reaches U62.6 (A0)
- net ##210: now also U101.23 (1Q), U58.5 (A0), U59.6 (A0), U60.6 (A0), U61.5 (A0), U63.6 (A0), U79.23 (1Q), U86.23 (1Q), U87.23 (1Q)
- net ##211: now reaches U62.7 (A1)
- net ##211: now also U101.22 (2Q), U58.7 (A1), U59.7 (A1), U60.7 (A1), U61.7 (A1), U63.7 (A1), U79.22 (2Q), U86.22 (2Q), U87.22 (2Q)
- net ##212: now reaches U62.8 (A2)
- net ##212: now also U101.21 (3Q), U58.6 (A2), U59.8 (A2), U60.8 (A2), U61.6 (A2), U63.8 (A2), U79.21 (3Q), U86.21 (3Q), U87.21 (3Q)
- net ##213: now reaches U62.9 (A3)
- net ##213: now also U101.20 (4Q), U58.12 (A3), U59.9 (A3), U60.9 (A3), U61.12 (A3), U63.9 (A3), U79.20 (4Q), U86.20 (4Q), U87.20 (4Q)
- net ##252: now reaches U55.2 (A12)
- net ##252: now also U54.2 (A12), U74.41 (A13), U86.5 (4D), U99.7 (6D)
- net ##250: now reaches U55.21 (A10)
- net ##250: now also U54.21 (A10), U74.39 (A11), U86.3 (2D), U99.5 (4D)
- net ##251: now reaches U55.23 (A11)
- net ##251: now also U54.23 (A11), U74.40 (A12), U86.4 (3D), U99.6 (5D)
- net ##249: now reaches U55.24 (A9)
- net ##249: now also U54.24 (A9), U74.38 (A10), U86.2 (1D), U99.4 (3D)
- net ##248: now reaches U55.25 (A8)
- net ##248: now also U54.25 (A8), U74.37 (A9), U79.10 (9D), U79.11 (10D), U99.3 (2D)
- net ##253: now reaches U55.26 (A13)
- net ##253: now also U54.26 (A13), U74.42 (A14), U86.6 (5D), U99.8 (7D)
- net ##247: now reaches U55.3 (A7)
- net ##247: now also U54.3 (A7), U74.36 (A8), U79.9 (8D), U99.2 (1D)
- net ##246: now reaches U55.4 (A6)
- net ##246: now also U119.6 (I6), U54.4 (A6), U74.35 (A7), U79.8 (7D), U81.9 (8D)
- net ##245: now reaches U55.5 (A5)
- net ##245: now also U119.7 (I7), U54.5 (A5), U74.34 (A6), U79.7 (6D), U81.8 (7D), U94.5 (E2)
- net ##244: now reaches U55.6 (A4)
- net ##244: now also U119.8 (I8), U54.6 (A4), U74.33 (A5), U79.6 (5D), U81.7 (6D)
- net ##243: now reaches U55.7 (A3)
- net ##243: now also U54.7 (A3), U74.32 (A4), U79.5 (4D), U81.6 (5D)
- net ##242: now reaches U55.8 (A2)
- net ##242: now also U134.6 (I6), U50.17 (A2), U54.8 (A2), U74.31 (A3), U79.4 (3D), U81.5 (4D), U94.3 (A2)
- net ##106: now reaches U67.15 (~{CAS})
- net ##106: now also U19.17 (~{CAS}), U20.17 (~{CAS}), U21.17 (~{CAS}), U22.17 (~{CAS}), U66.15 (~{CAS}), U75.17
- net ##111: now reaches U108.1 (~{OE})
- net ##111: now also U113.15 (O5)
- net ##228: now reaches U108.10 (9D)
- net ##228: now also U101.10 (9~{D}), U101.11 (10~{D}), U107.4 (3D), U108.11 (10D), U122.5 (I5), U84.17 (3~{Q}), RN1.8 (R7)
- net ##220: now reaches U108.2 (1D)
- net ##220: now also U100.4 (3D), U101.2 (1~{D}), U122.14 (O10), U99.17 (3~{Q})
- net ##221: now reaches U108.3 (2D)
- net ##221: now also U100.5 (4D), U101.3 (2~{D}), U122.13 (I12), U99.16 (4~{Q})
- net ##222: now reaches U108.4 (3D)
- net ##222: now also U100.6 (5D), U101.4 (3~{D}), U122.11 (I11), U99.15 (5~{Q})
- net ##223: now reaches U108.5 (4D)
- net ##223: now also U100.7 (6D), U101.5 (4~{D}), U122.10 (I10), U99.14 (6~{Q})
- net ##224: now reaches U108.6 (5D)
- net ##224: now also U100.8 (7D), U101.6 (5~{D}), U122.9 (I9), U99.13 (7~{Q})
- net ##225: now reaches U108.7 (6D)
- net ##225: now also U100.9 (8D), U101.7 (6~{D}), U122.8 (I8), U99.12 (8~{Q})
- net ##226: now reaches U108.8 (7D)
- net ##226: now also U101.8 (7~{D}), U107.2 (1D), U122.7 (I7), U84.19 (1~{Q})
- net ##227: now reaches U108.9 (8D)
- net ##227: now also U101.9 (8~{D}), U107.3 (2D), U122.6 (I6), U84.18 (2~{Q}), RN1.9 (R8)
- net ##254: now reaches U74.43 (A15)
- net ##254: now also U86.7 (6D), U99.9 (8D)
- net ##238: now reaches U99.18 (2~{Q})
- net ##238: now also U100.3 (2D), U102.10 (9D), U102.11 (10D), U122.18 (IO6), U87.10 (9~{D}), U87.11 (10~{D})
- net ##237: now reaches U99.19 (1~{Q})
- net ##237: now also U100.2 (1D), U102.9 (8D), U122.17 (IO7), U87.9 (8~{D})
- net ##110: now reaches U75.16
- net ##110: now also U113.18 (O2), U120.5, U75.19, U75.2
- net ##230: now reaches U87.2 (1~{D})
- net ##230: now also U102.2 (1D), U115.3 (2D), U81.18 (2~{Q})
- net ##231: now reaches U87.3 (2~{D})
- net ##231: now also U102.3 (2D), U115.4 (3D), U119.4 (I4), U81.17 (3~{Q})
- net ##232: now reaches U87.4 (3~{D})
- net ##232: now also U102.4 (3D), U115.5 (4D), U119.3 (I3), U81.16 (4~{Q})
- net ##233: now reaches U87.5 (4~{D})
- net ##233: now also U102.5 (4D), U115.6 (5D), U81.15 (5~{Q})
- net ##234: now reaches U87.6 (5~{D})
- net ##234: now also U102.6 (5D), U115.7 (6D), U81.14 (6~{Q})
- net ##235: now reaches U87.7 (6~{D})
- net ##235: now also U102.7 (6D), U115.8 (7D), U119.2 (I2), U81.13 (7~{Q})
- net ##236: now reaches U87.8 (7~{D})
- net ##236: now also U102.8 (7D), U115.9 (8D), U122.16 (IO8), U81.12 (8~{Q})
- new net VCC: RN1.1 (common)
- no-connect marks 0 -> 1

Commit message: AP: Lots more tracing
Parts:
- added RP4, RP5, RP6, RP7, RP8, RP9: R_Network09_US, Resistor_THT:R_Array_SIP10, symbol Device:R_Network09_US
- renumbered RN1 to RP11
Connections:
- net VCC: now also RP6.1 (common), RP7.1 (common), RP8.1 (common)
- net ##150: now reaches U83.17 (IO7)
- net ##150: now also U121.8 (I8), U54.22 (~{OE}), U55.22 (~{OE})
- net ##155: now reaches U83.2 (I2)
- net ##155: now also U119.5 (I5), U121.5 (I5), U135.2 (D), U74.6 (AS), U94.4 (E1)
- net ##123: now reaches U11.3 (~{W})
- net ##123: now also U1.3 (~{W}), U10.3 (~{W}), U12.3 (~{W}), U13.3 (~{W}), U14.3 (~{W}), U15.3 (~{W}), U16.3 (~{W}), U17.3 (~{W}), U18.3 (~{W}), U2.3 (~{W}), U3.3 (~{W}), U4.3 (~{W}), U5.3 (~{W}), U6.3 (~{W}), U7.3 (~{W}), U8.3 (~{W}), U9.3 (~{W}), U96.5 (O2a)
- net ##115: now reaches U11.4 (~{RAS})
- net ##115: now also U10.4 (~{RAS}), U12.4 (~{RAS}), U120.3, U13.4 (~{RAS}), U14.4 (~{RAS}), U15.4 (~{RAS}), U16.4 (~{RAS}), U17.4 (~{RAS}), U18.4 (~{RAS}), U36.4 (~{RAS}), U37.4 (~{RAS}), U38.4 (~{RAS}), U39.4 (~{RAS}), U40.4 (~{RAS}), U41.4 (~{RAS}), U42.4 (~{RAS}), U43.4 (~{RAS}), U44.4 (~{RAS})
- net ##122: now reaches U30.3 (~{W})
- net ##122: now also U27.3 (~{W}), U28.3 (~{W}), U29.3 (~{W}), U31.3 (~{W}), U32.3 (~{W}), U33.3 (~{W}), U34.3 (~{W}), U35.3 (~{W}), U36.3 (~{W}), U37.3 (~{W}), U38.3 (~{W}), U39.3 (~{W}), U40.3 (~{W}), U41.3 (~{W}), U42.3 (~{W}), U43.3 (~{W}), U44.3 (~{W}), U96.9 (O4a)
- net ##116: now reaches U30.4 (~{RAS})
- net ##116: now also U1.4 (~{RAS}), U2.4 (~{RAS}), U27.4 (~{RAS}), U28.4 (~{RAS}), U29.4 (~{RAS}), U3.4 (~{RAS}), U31.4 (~{RAS}), U32.4 (~{RAS}), U33.4 (~{RAS}), U34.4 (~{RAS}), U35.4 (~{RAS}), U4.4 (~{RAS}), U5.4 (~{RAS}), U6.4 (~{RAS}), U7.4 (~{RAS}), U75.11, U8.4 (~{RAS}), U9.4 (~{RAS})
- net GND: now reaches U48.16 (~{OE})
- net GND: now also U19.16 (~{OE}), U20.16 (~{OE}), U21.16 (~{OE}), U22.16 (~{OE}), U45.16 (~{OE}), U46.16 (~{OE}), U47.16 (~{OE}), U59.16 (~{OE}), U60.16 (~{OE}), U62.16 (~{OE}), U63.16 (~{OE}), RP9.1 (common)
- net ##120: now reaches U48.3 (~{WE})
- net ##120: now also U21.3 (~{WE}), U22.3 (~{WE}), U47.3 (~{WE}), U65.3 (~{W}), U67.3 (~{W}), U96.7 (O3a)
- net ##114: now reaches U48.4 (~{RAS})
- net ##114: now also U45.4 (~{RAS}), U46.4 (~{RAS}), U47.4 (~{RAS}), U64.4 (~{RAS}), U65.4 (~{RAS}), U75.9
- net ##177: now reaches U111.21 (~{WR})
- net ##177: now also U121.11 (I10), U126.6 (I6), U127.9 (I9), U133.21 (~{WR}), U49.1 (DIR), U53.13 (R/~{W}), U72.1 (DIR), U74.9 (R/W), U90.21 (~{WR})
- net ##131: now reaches U111.3 (~{CD_{A}})
- net ##131: now also U111.39 (~{CTS_{A}}), U111.5 (~{CD_{B}}), U111.6 (~{CTS_{B}}), U113.11 (~{OE}), U93.11 (~{OE}), RP9.6 (R5)
- net ##118: now reaches U62.3 (~{WE})
- net ##118: now also U110.18 (O0a), U61.3 (~{W}), U63.3 (~{WE})
- net ##112: now reaches U62.4 (~{RAS})
- net ##112: now also U110.12 (O3a), U58.4 (~{RAS}), U59.4 (~{RAS}), U60.4 (~{RAS}), U61.4 (~{RAS}), U63.4 (~{RAS})
- net ##149: now reaches U55.20 (~{CE})
- net ##149: now also U110.1 (OEa), U110.19 (OEb), U116.19 (OEb), U118.15 (OE), U129.12, U129.3, U130.11 (2~{OE}), U130.2 (1~{OE}), U133.29 (~{IPI}/RxDRQ_{B}), U137.2, U137.5, U50.15 (~{E}1), U50.16 (~{E}0), U54.20 (~{CE}), U96.1 (OEa), U97.13 (~{OE})
- net ##113: now reaches U67.4 (~{RAS})
- net ##113: now also U19.4 (~{RAS}), U20.4 (~{RAS}), U21.4 (~{RAS}), U22.4 (~{RAS}), U66.4 (~{RAS}), U75.6
- net ##187: now reaches U108.13 (LE)
- net ##187: now also U101.13 (LE), U102.13 (LE), U104.12 (STT), U104.8 (STR), U125.10 (CET), U125.7 (CEP), U128.10 (CET), U128.7 (CEP), U139.10 (CET), U139.7 (CEP), U140.10 (CET), U140.7 (CEP), U50.13 (E3), U50.14 (E2), U76.10 (CET), U76.7 (CEP), U76.9 (~{PE}), U79.13 (LE), U85.12 (STT), U85.8 (STR), U86.13 (LE), U87.13 (LE), U97.1 (~{PL}), RP5.7 (R6)
- net ##159: now reaches U89.1 (OE)
- net ##159: now also U134.11 (~{OE}), U95.4 (I4), RP9.4 (R3)
- net ##156: now reaches U140.14 (Q0)
- net ##156: now also U130.14 (2CLK), U135.3 (C), U138.13
- net ##121: now reaches U45.3 (~{WE})
- net ##121: now also U19.3 (~{WE}), U20.3 (~{WE}), U46.3 (~{WE}), U64.3 (~{W}), U66.3 (~{W}), U96.3 (O1a)
- net ##176: now reaches U49.19 (~{OE})
- net ##176: now also U136.19 (O1)
- net ##126: now reaches U93.1 (CLK)
- net ##126: now also U105.1 (CLK), U112.1 (CLK), U113.1 (CLK), U127.1 (CLK), U130.23 (1CLK), U135.11 (C), U138.12
- net ##127: now reaches U93.4 (I4)
- net ##127: now also U113.19 (IO1), U120.11
- net ##173: now reaches U93.5 (I5)
- net ##173: now also U112.2 (I2), U127.14 (O6), U23.24 (~{OE}), U80.24 (~{OE})
- net ##175: now reaches U70.1 (DIR)
- net ##175: now also U136.17 (IO3), U51.1 (DIR), U52.1 (DIR)
- net ##179: now reaches U70.19 (~{OE})
- net ##179: now also U136.16 (IO4)
- net ##192: now reaches U74.23 (IPL2)
- net ##192: now also U68.17 (O3), RP8.3 (R2)
- net ##193: now reaches U74.24 (IPL1)
- net ##193: now also U68.16 (O4), RP8.4 (R3)
- net ##194: now reaches U74.25 (IPL0)
- net ##194: now also U68.15 (O5), RP8.5 (R4)
- net ##186: now reaches U134.12 (IO8)
- net ##186: now also U50.4 (~{OE}0), U50.5 (~{OE}1)
- net ##197: now reaches U134.14 (O6)
- net ##197: now also U68.1 (CLK), U78.9 (Cp)
- net ##188: now reaches U109.5 (B)
- net ##188: now also U109.13 (A), U109.9 (B), U114.13 (I1b), U114.2 (I0a), U116.2 (I0a), U117.12 (B), U117.5 (B), U117.9 (B), U131.5 (4D), U131.9 (8D), U50.12 (P), U71.19 (A8), U88.5 (B), U88.9 (B), RP5.10 (R9)
- net ##160: now reaches RP11.7 (R6)
- net ##160: now also U107.5 (4D), U122.4 (I4), U84.16 (4~{Q}), U95.5 (I5)
- net ##145: now reaches U90.3 (~{CD_{A}})
- net ##145: now also U105.11 (~{OE}), U112.11 (~{OE}), U68.11 (~{OE}), U90.39 (~{CTS_{A}}), U90.5 (~{CD_{B}}), U90.6 (~{CTS_{B}}), RP9.5 (R4)
- net ##196: now reaches U68.12 (IO8)
- net ##196: now also U78.7 (Q2)
- net ##195: now reaches U68.13 (IO7)
- net ##195: now also U78.5 (Q1)
- net ##171: now reaches U68.18 (IO2)
- net ##171: now also U23.1 (T/~{R})
- net ##191: now reaches U68.19 (IO1)
- net ##191: now also U78.15 (Q5)
- net ##185: now reaches U68.2 (I2)
- net ##185: now also U50.11 (Q7), RP6.4 (R3)
- net ##184: now reaches U68.3 (I3)
- net ##184: now also U50.9 (Q6), RP6.5 (R4)
- net ##183: now reaches U68.4 (I4)
- net ##183: now also U50.8 (Q5), RP6.6 (R5)
- net ##182: now reaches U68.5 (I5)
- net ##182: now also U50.18 (Q4), RP6.7 (R6)
- net ##181: now reaches U68.6 (I6)
- net ##181: now also U50.19 (Q3), RP6.8 (R7)
- net ##180: now reaches U68.7 (I7)
- net ##180: now also U50.1 (Q2), RP6.9 (R8)
- net ##189: now reaches U68.8 (I8)
- net ##189: now also U110.4 (I1a), U127.19 (IO1)
- net ##190: now reaches U68.9 (I9)
- net ##190: now also U78.10 (Q3)
- net ##154: now reaches U120.1
- net ##154: now also U120.4, U95.14 (O10)
- net ##117: now reaches U120.2
- net ##117: now also U113.17 (O3), U75.13, U75.5, U75.8
- net ##174: now reaches U136.14 (IO6)
- net ##174: now also U51.19 (~{OE})
- net ##178: now reaches U136.15 (IO5)
- net ##178: now also U52.19 (~{OE})
- net ##132: now reaches U136.5 (I5)
- net ##132: now also U105.2 (I2), U113.2 (I2), U116.9 (O0b), U127.3 (I3), U24.1 (T/~{R}), U25.1 (T/~{R}), U26.1 (T/~{R}), U95.11 (I11)
- net ##164: now reaches U136.6 (I6)
- net ##164: now also U116.7 (O1b), U127.4 (I4), U95.9 (I9)
- net ##163: now reaches U136.7 (I7)
- net ##163: now also U115.2 (1D), U127.5 (I5), U81.19 (1~{Q}), U95.8 (I8)
- net ##161: now reaches U114.4 (I1a)
- net ##161: now also U95.6 (I6), W2.4 (Pin_4), RP8.8 (R7)
- net ##162: now reaches U114.6 (I2a)
- net ##162: now also U95.7 (I7), RP8.10 (R9)
- net ##152: now reaches U75.15
- net ##152: now also U75.7, U95.17 (IO7)
- net ##153: now reaches U75.1
- net ##153: now also U75.12, U95.16 (IO8)
- net ##151: now reaches U75.4
- net ##151: now also U75.18, U95.18 (IO6)
- net ##143: now reaches U130.20 (1Q3)
- net ##143: now also U105.8 (I8), U112.6 (I6), U125.2 (CP), U128.2 (CP)
- net ##134: now reaches U130.22 (1Q1)
- net ##134: now also U105.4 (I4), U113.4 (I4), U127.13 (IO7)
- net ##165: now reaches U130.7 (2D1)
- net ##165: now also U116.15 (I2b), U116.16 (O1a), U95.10 (I10), RP7.9 (R8)
- net ##130: now reaches U137.8
- net ##130: now also U121.17 (IO3), U129.6, U96.13 (O6b)
- net ##119: now reaches U59.3 (~{WE})
- net ##119: now also U110.16 (O1a), U58.3 (~{W}), U60.3 (~{WE})
- net ##158: now reaches U122.19 (IO5)
- net ##158: now also U95.3 (I3)
- net ##157: now reaches U122.22 (O2)
- net ##157: now also U95.2 (I2)
- net ##170: now reaches U23.11 (ODD/~{EVEN})
- net ##170: now also U24.11 (ODD/~{EVEN}), U25.11 (ODD/~{EVEN}), U26.11 (ODD/~{EVEN}), U80.11 (ODD/~{EVEN}), U97.20 (03)
- net ##172: now reaches U23.12 (~{ERROR})
- net ##172: now also U112.3 (I3), RP7.4 (R3)
- net ##128: now reaches U102.1 (~{OE})
- net ##128: now also U113.14 (O6)
- net ##147: now reaches U128.1 (~{MR})
- net ##147: now also U105.13 (O7), U95.13 (I12)
- net ##144: now reaches U128.15 (TC)
- net ##144: now also U105.9 (I9)
- net ##148: now reaches U105.12 (O8)
- net ##148: now also U96.15 (OEb)
- net ##146: now reaches U105.14 (O6)
- net ##146: now also U96.12 (I5)
- net ##140: now reaches U105.15 (O5)
- net ##140: now also U113.9 (I9)
- net ##139: now reaches U105.16 (O4)
- net ##139: now also U113.8 (I8)
- net ##138: now reaches U105.17 (O3)
- net ##138: now also U113.7 (I7)
- net ##137: now reaches U105.18 (O2)
- net ##137: now also U113.6 (I6)
- net ##135: now reaches U105.19 (O1)
- net ##135: now also U113.5 (I5)
- net ##133: now reaches U105.3 (I3)
- net ##133: now also U113.3 (I3), U95.15 (IO9)
- net ##141: now reaches U105.5 (I5)
- net ##141: now also U24.12 (~{ERROR}), U25.12 (~{ERROR}), RP7.2 (R1)
- net ##142: now reaches U105.6 (I6)
- net ##142: now also U26.12 (~{ERROR}), RP7.3 (R2)
- net ##169: now reaches U106.9 (I9)
- net ##169: now also U129.8, U131.3 (2D), U96.11 (O5b), RP4.5 (R4)
- net ##168: now reaches U26.24 (~{OE})
- net ##168: now also U95.19 (IO5)
- net ##125: now reaches U96.10 (I4)
- net ##125: now also U95.22 (IO2), U96.6 (I3)
- net ##129: now reaches U96.14 (I6)
- net ##129: now also U113.13 (O7)
- net ##124: now reaches U96.2 (I1)
- net ##124: now also U95.23 (O1), U96.4 (I2)
- net ##167: now reaches U95.20 (IO4)
- net ##167: now also U24.24 (~{OE})
- net ##166: now reaches U95.21 (IO3)
- net ##166: now also U25.24 (~{OE})
- no-connect marks 1 -> 8
