File: attachment_processor_4/attachment_processor_4.kicad_sch (KiCad schematic)
At the start: 150 parts, among them U1 TMS4256, U10 TMS4256, U100 74ALS576, U101 74ALS842, U102 74ALS841, U103 MC1488, U104 WD1943-PD, U105 TIBPAL16R8, U106 PAL16P8, U107 74ALS576, U108 74ALS841, U109 MC1488, U11 TMS4256, U110 74ALS244, U111 P8274, U112 TIBPAL16R8, U113 TIBPAL16R6, U114 74ALS240, U115 74ALS576, U116 74ALS240, U117 MC1488, U118 74ALS257, U119 PAL16L8, U12 TMS4256, U120 74ALS832, U121 TIBPAL16L8, U122 PAL20L8, U124 MC1489, U125 74ALS161, U126 PAL16R4, U127 TIBPAL16R4, U128 74ALS161, U129 74LS125, U13 TMS4256, U130 74ALS874, U131 74AS576, U132 74ALS257, U133 P8274, U134 PAL16R6, U135 74AS74, U136 PAL16L8, U137 74LS125, U138 74AS1004, U139 74AS161, U14 TMS4256, U140 74AS161, U15 TMS4256, U16 TMS4256, U17 TMS4256, U18 TMS4256, U19 MB81C4256, U2 TMS4256, U20 MB81C4256, U21 MB81C4256, U22 MB81C4256, U23 74F657, U24 74F657, U25 74F657, U26 74F657, U27 TMS4256, U28 TMS4256, U29 TMS4256, U3 TMS4256, U30 TMS4256, U31 TMS4256, U32 TMS4256, U33 TMS4256, U34 TMS4256, U35 TMS4256, U36 TMS4256, U37 TMS4256, U38 TMS4256, U39 TMS4256, U4 TMS4256, U40 TMS4256, U41 TMS4256, U42 TMS4256, U43 TMS4256, U44 TMS4256, U45 MB81C4256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

Commit message: AP: more tracing
Parts:
- added J1: Conn_02x49_Odd_Even, symbol custom:Conn_02x49_Odd_Even
- added R1, R2, R3, R4, R5, R6, R7: R, symbol Device:R
- added RP10: R_Network09_US, Resistor_THT:R_Array_SIP10, symbol Device:R_Network09_US
- added U98: TL7705A, symbol Power_Supervisor:TL7705A
Connections:
- net ##157: now also U122.20 (IO4); no longer U122.22 (O2)
- net ##165: now also J1.38 (Pin_38)
- net GND: now also W3.2 (Pin_2), W3.3 (Pin_3)
- net VCC: now also R1.1
- net ##354: now reaches U83.23 (O1)
- net ##354: now also U92.1 (~{Mr}), U97.16 (O7), J1.45 (Pin_45)
- net ##337: now reaches U138.1
- net ##337: now also U126.1 (CLK), U138.5, U140.12 (Q2), U74.15 (CLK), U77.11 (C), R5.2
- net ##332: now reaches U138.2
- net ##332: now also U77.3 (C)
- net ##349: now reaches U111.2 (~{RESET})
- net ##349: now also U106.7 (I7), U110.3 (O3b), U133.2 (~{RESET}), U90.2 (~{RESET}), U97.9 (I7), J1.41 (Pin_41)
- net ##370: now reaches U111.22 (~{RD})
- net ##370: now also U116.8 (I3a), U126.13 (IO7), U133.22 (~{RD}), U90.22 (~{RD})
- net ##321: now reaches U111.28 (~{INT})
- net ##321: now also U133.28 (~{INT}), U78.4 (D1), U90.28 (~{INT}), RP10.2 (R1)
- net ##346: now reaches U140.1 (~{MR})
- net ##346: now also RP7.7 (R6), U139.1 (~{MR}), U97.3 (I1), U98.5 (~{RESET})
- net ##361: now reaches U94.10 (O5)
- net ##361: now also U106.4 (I4)
- net ##317: now reaches U94.11 (O4)
- net ##317: now also U69.11 (Cp)
- net ##387: now reaches U94.13 (O2)
- net ##387: now also U121.14 (IO6)
- net ##350: now reaches U94.15 (O0)
- net ##350: now also U97.10 (I8)
- net ##343: now reaches U94.7 (O7)
- net ##343: now also U100.1 (~{OE}), U115.1 (~{OE})
- net ##359: now reaches U94.9 (O6)
- net ##359: now also U107.1 (~{OE}), U131.1 (~{OE})
- net ##384: now reaches U93.12 (O8)
- net ##384: now also U121.9 (I9)
- net ##328: now reaches U93.16 (O4)
- net ##328: now also U79.1 (~{OE})
- net ##330: now reaches U93.17 (O3)
- net ##330: now also U86.1 (~{OE})
- net ##329: now reaches U93.18 (O2)
- net ##329: now also U87.1 (~{OE})
- net ##342: now reaches U93.19 (O1)
- net ##342: now also U101.1 (~{OE})
- net ##388: now reaches U74.10 (DTACK)
- net ##388: now also U121.12 (O8)
- net ##386: now reaches U74.22 (BERR)
- net ##386: now also U121.15 (IO5)
- net ##360: now reaches U134.13 (O7)
- net ##360: now also U106.2 (I2)
- net ##382: now reaches U134.15 (O5)
- net ##382: now also U121.6 (I6)
- net ##366: now reaches RP11.10 (R9)
- net ##366: now also U114.15 (I2b), W3.4 (Pin_4)
- net ##307: now reaches RP11.2 (R1)
- net ##307: now also U121.13 (IO7), U71.15 (~{CE}), J1.9 (Pin_9)
- net ##358: now reaches RP11.3 (R2)
- net ##358: now also U107.9 (8D), U122.23 (O1), U84.12 (8~{Q}), J1.82 (Pin_82)
- net ##357: now reaches RP11.4 (R3)
- net ##357: now also U107.8 (7D), U122.1 (I1), U84.13 (7~{Q}), J1.81 (Pin_81)
- net ##356: now reaches RP11.5 (R4)
- net ##356: now also U107.7 (6D), U122.2 (I2), U84.14 (6~{Q}), J1.80 (Pin_80)
- net ##355: now reaches RP11.6 (R5)
- net ##355: now also U107.6 (5D), U122.3 (I3), U84.15 (5~{Q}), J1.79 (Pin_79)
- net ##331: now reaches U76.1 (~{MR})
- net ##331: now also U116.5 (O2b), U119.11 (I10), U121.3 (I3), U77.2 (D)
- net ##339: now reaches U76.15 (TC)
- net ##339: now also U106.1 (I1)
- net ##338: now reaches U76.2 (CP)
- net ##338: now also U106.11 (I10), U130.8 (2D2), U139.13 (Q1), R2.2
- net ##308: now reaches U136.18 (IO2)
- net ##308: now also U72.19 (~{OE})
- net ##327: now reaches U136.3 (I3)
- net ##327: now also U106.3 (I3), U116.1 (OEa), U121.4 (I4), U137.1, U137.4, U77.12 (D), U81.1 (~{OE}), U81.11 (LE), U84.1 (~{OE}), U84.11 (LE), U99.1 (~{OE}), U99.11 (LE)
- net ##325: now reaches U135.1 (~{R})
- net ##325: now also RP5.8 (R7), U128.9 (~{PE}), U130.1 (1~{CLR}), U130.13 (2~{CLR}), U135.13 (~{R}), U77.1 (~{R}), U77.13 (~{R}), U78.1 (~{Mr})
- net ##333: now reaches U135.4 (~{S})
- net ##333: now also RP5.9 (R8), U125.9 (~{PE}), U135.10 (~{S}), U77.4 (~{S})
- net ##368: now reaches U114.1 (OEa)
- net ##368: now also U114.19 (OEb), U121.19 (O1)
- net ##352: now reaches U114.11 (I0b)
- net ##352: now also U97.21 (O2)
- net ##367: now reaches U114.17 (I3b)
- net ##367: now also RP8.6 (R5), W3.1 (Pin_1)
- net ##365: now reaches U114.8 (I3a)
- net ##365: now also J?.12 (Pin_12), J?.15 (Pin_15)
- net ##318: now reaches U69.1 (OE)
- net ##318: now also RP9.3 (R2), U126.11 (~{OE}), U127.11 (~{OE})
- net ##313: now reaches U69.12 (O4)
- net ##313: now also U85.4 (RA)
- net ##314: now reaches U69.15 (O5)
- net ##314: now also U85.5 (RB)
- net ##315: now reaches U69.16 (O6)
- net ##315: now also U85.6 (RC)
- net ##316: now reaches U69.19 (O7)
- net ##316: now also U85.7 (RD)
- net ##309: now reaches U69.2 (O0)
- net ##309: now also U85.16 (TA)
- net ##310: now reaches U69.5 (O1)
- net ##310: now also U85.15 (TB)
- net ##311: now reaches U69.6 (O2)
- net ##311: now also U85.14 (TC)
- net ##312: now reaches U69.9 (O3)
- net ##312: now also U85.13 (TD)
- net ##378: now reaches U129.11
- net ##378: now also U131.6 (5D), J1.10 (Pin_10)
- net ##334: now reaches U77.6 (~{Q})
- net ##334: now also U126.8 (I8)
- net ##379: now reaches U137.3
- net ##379: now also U120.13, U131.7 (6D), J1.11 (Pin_11)
- net ##345: now reaches U139.11 (Q3)
- net ##345: now also U97.2 (I0)
- net ##344: now reaches U100.11 (CLK)
- net ##344: now also U106.13 (IO7), U107.11 (CLK), U115.11 (CLK), U131.11 (CLK)
- net ##377: now reaches U122.15 (O9)
- net ##377: now also U119.1 (I1)
- net ##375: now reaches U122.21 (IO3)
- net ##375: now also U127.2 (I2)
- net ##341: now reaches U85.17 (fT)
- net ##341: now also U110.11 (I0b)
- net ##340: now reaches U85.3 (fR)
- net ##340: now also U110.13 (I1b)
- net ##369: now reaches U126.16 (O4)
- net ##369: now also U116.6 (I2a)
- net ##326: now reaches U126.17 (O3)
- net ##326: now also U81.2 (1D)
- net ##336: now reaches U126.18 (IO2)
- net ##336: now also U77.10 (~{S})
- net ##374: now reaches U126.7 (I7)
- net ##374: now also U116.3 (O3b)
- net ##362: now reaches U110.2 (I0a)
- net ##362: now also U106.5 (I5), U127.18 (IO2)
- net ##323: now reaches U78.11 (D3)
- net ##323: now also U106.17 (IO3)
- net ##324: now reaches U78.14 (D5)
- net ##324: now also U97.18 (O5)
- net ##322: now reaches U78.6 (D2)
- net ##322: now also U53.9 (~{IRQ}), R1.2
- net ##371: now reaches U116.11 (I0b)
- net ##371: now also U116.12 (O3a), J1.37 (Pin_37)
- net ##372: now reaches U116.13 (I1b)
- net ##372: now also U116.14 (O2a), J1.40 (Pin_40)
- net ##373: now reaches U116.17 (I3b)
- net ##373: now also U116.18 (O0a), J1.33 (Pin_33)
- net ##335: now reaches U116.4 (I1a)
- net ##335: now also U77.8 (~{Q})
- net ##364: now reaches U106.14 (IO6)
- net ##364: now also U121.2 (I2), U131.2 (1D)
- net ##319: now reaches U106.19 (O1)
- net ##319: now also U80.1 (T/~{R})
- net ##363: now reaches U106.8 (I8)
- net ##363: now also U112.13 (O7), U131.4 (3D)
- net ##381: now reaches U121.1 (I1)
- net ##381: now also U119.19 (O1)
- net ##351: now reaches U121.16 (IO4)
- net ##351: now also U97.11 (I9)
- net ##385: now reaches U121.18 (IO2)
- net ##385: now also U129.4, U129.5
- net ##383: now reaches U121.7 (I7)
- net ##383: now also U119.12 (O8)
- net ##320: now reaches U112.4 (I4)
- net ##320: now also U80.12 (~{ERROR})
- net ##380: now reaches U120.12
- net ##380: now also U131.8 (7D), U137.6, J1.12 (Pin_12)
- net ##198: now reaches U71.1 (A0)
- net ##198: now also U97.6 (I4), J1.13 (Pin_13)
- net ##304: now reaches U71.16 (A5)
- net ##304: now also J1.18 (Pin_18)
- net ##305: now reaches U71.17 (A6)
- net ##305: now also J1.19 (Pin_19)
- net ##306: now reaches U71.18 (A7)
- net ##306: now also J1.20 (Pin_20)
- net ##199: now reaches U71.2 (A1)
- net ##199: now also J1.14 (Pin_14)
- net ##301: now reaches U71.3 (A2)
- net ##301: now also J1.15 (Pin_15)
- net ##302: now reaches U71.4 (A3)
- net ##302: now also J1.16 (Pin_16)
- net ##303: now reaches U71.5 (A4)
- net ##303: now also J1.17 (Pin_17)
- net ##347: now reaches U119.17 (IO3)
- net ##347: now also U97.7 (I5)
- net ##348: now reaches U119.18 (IO2)
- net ##348: now also U97.8 (I6)
- net ##353: now reaches U97.19 (O4)
- net ##353: now also J1.46 (Pin_46)
- new net ##376: J1.32 (Pin_32), U122.22 (O2)
- no-connect marks 8 -> 31
Other:
- moved on the sheet: U129A, U129B, U129C, U135B, U137A, U137B, U137C, U138A, U138B, U138C, U77A

Commit message: AP: basically done tracing, only thing left are rs232 related and some passives
Parts:
- added RP3: R_Network09_US, Resistor_THT:R_Array_SIP10, symbol Device:R_Network09_US
- added U123: CXO_DIP14, Oscillator:Oscillator_DIP-14, symbol Oscillator:CXO_DIP14
Connections:
- net ##130: now also J1.39 (Pin_39), RP6.3 (R2)
- net ##159: now also U132.15 (OE)
- net ##160: now also J1.76 (Pin_76)
- net ##163: now also J1.57 (Pin_57)
- net ##169: now also J1.3 (Pin_3)
- net ##170: now also J1.52 (Pin_52)
- net ##180: now also J1.49 (Pin_49)
- net ##181: now also J1.50 (Pin_50)
- net ##182: now also J1.51 (Pin_51)
- net ##183: now also J1.4 (Pin_4)
- net ##184: now also J1.5 (Pin_5)
- net ##185: now also J1.6 (Pin_6)
- net ##186: now also J1.8 (Pin_8)
- net ##197: now also J1.7 (Pin_7)
- net ##220: now also J1.67 (Pin_67)
- net ##221: now also J1.68 (Pin_68)
- net ##222: now also J1.69 (Pin_69)
- net ##223: now also J1.70 (Pin_70)
- net ##224: now also J1.71 (Pin_71)
- net ##225: now also J1.72 (Pin_72)
- net ##226: now also J1.73 (Pin_73)
- net ##227: now also J1.74 (Pin_74)
- net ##228: now also J1.75 (Pin_75)
- net ##230: now also J1.58 (Pin_58)
- net ##231: now also J1.59 (Pin_59)
- net ##232: now also J1.60 (Pin_60)
- net ##233: now also J1.61 (Pin_61)
- net ##234: now also J1.62 (Pin_62)
- net ##235: now also J1.63 (Pin_63)
- net ##236: now also J1.64 (Pin_64)
- net ##237: now also J1.65 (Pin_65)
- net ##238: now also J1.66 (Pin_66)
- net ##242: now also U126.9 (I9)
- net ##327: now also U126.14 (O6), U129.13
- net ##73: now also J1.21 (Pin_21), RP5.4 (R3)
- net ##74: now also J1.22 (Pin_22)
- net ##75: now also J1.23 (Pin_23)
- net ##76: now also J1.24 (Pin_24)
- net ##77: now also J1.25 (Pin_25)
- net ##78: now also J1.26 (Pin_26)
- net ##79: now also J1.27 (Pin_27)
- net ##80: now also J1.28 (Pin_28)
- net GND: now also J1.1 (Pin_1), J1.2 (Pin_2), J1.29 (Pin_29), J1.30 (Pin_30), J1.53 (Pin_53), J1.54 (Pin_54), J1.77 (Pin_77), J1.78 (Pin_78), J1.97 (Pin_97), J1.98 (Pin_98), U129.2, U123.1 (EN)
- net VCC: now also J1.55 (Pin_55), J1.56 (Pin_56), J1.91 (Pin_91), J1.92 (Pin_92)
- net ##410: now reaches U83.15 (O9)
- net ##410: now also U94.6 (E3)
- net ##438: now reaches U83.16 (IO8)
- net ##438: now also U119.9 (I9)
- net ##427: now reaches U83.19 (IO5)
- net ##427: now also U127.8 (I8)
- net ##424: now reaches U83.20 (IO4)
- net ##424: now also U134.9 (I9), U136.9 (I9)
- net ##423: now reaches U83.21 (IO3)
- net ##423: now also U136.8 (I8)
- net ##434: now reaches U83.22 (O2)
- net ##434: now also U126.4 (I4)
- net ##453: now reaches U83.3 (I3)
- net ##453: now also U74.26 (FC2)
- net ##452: now reaches U83.4 (I4)
- net ##452: now also U74.27 (FC1)
- net ##451: now reaches U83.5 (I5)
- net ##451: now also U74.28 (FC0)
- net ##398: now reaches U111.1 (CLK)
- net ##398: now also U133.1 (CLK), U134.1 (CLK), U134.5 (I5), U139.2 (CP), U140.11 (Q3), U90.1 (CLK)
- net ##436: now reaches U111.23 (~{CS})
- net ##436: now also U119.15 (IO5)
- net ##433: now reaches U111.27 (~{INTA})
- net ##433: now also U133.27 (~{INTA}), U134.17 (O3), U90.27 (~{INTA})
- net ##411: now reaches U89.11 (Cp)
- net ##411: now also U94.12 (O3)
- net ##400: now reaches U140.13 (Q1)
- net ##400: now also U138.3
- net ##399: now reaches U140.2 (CP)
- net ##399: now also U123.8 (OUT)
- net ##397: now reaches U140.9 (~{PE})
- net ##397: now also RP5.6 (R5), U139.9 (~{PE})
- net ##420: now reaches U132.1 (S)
- net ##420: now also U118.1 (S), U92.19 (Q7)
- net ##412: now reaches U94.14 (O1)
- net ##412: now also U92.11 (Cp)
- net ##409: now reaches U93.13 (O7)
- net ##409: now also U137.9
- net ##441: now reaches U93.14 (O6)
- net ##441: now also U110.6 (I2a), U112.7 (I7), U125.1 (~{MR})
- net ##447: now reaches U93.15 (O5)
- net ##447: now also U110.8 (I3a)
- net ##428: now reaches U93.2 (I2)
- net ##428: now also U127.16 (O4)
- net ##421: now reaches U93.3 (I3)
- net ##421: now also U112.5 (I5), U127.15 (O5), U136.1 (I1)
- net ##443: now reaches U93.6 (I6)
- net ##443: now also U112.19 (O1)
- net ##444: now reaches U93.7 (I7)
- net ##444: now also U112.18 (O2)
- net ##445: now reaches U93.8 (I8)
- net ##445: now also U112.17 (O3)
- net ##446: now reaches U93.9 (I9)
- net ##446: now also U112.16 (O4)
- net ##456: now reaches U74.12 (BGACK)
- net ##456: now also U74.13 (BR), RP3.2 (R1)
- net ##425: now reaches U74.17 (HALT)
- net ##425: now also RP8.2 (R1), U136.13 (IO7)
- net ##426: now reaches U74.18 (RESET)
- net ##426: now also RP8.7 (R6), U110.15 (I2b), U110.17 (I3b), U136.12 (O8)
- net ##455: now reaches U74.19 (VMA)
- net ##455: now also U53.15 (~{CS_{0}})
- net ##454: now reaches U74.20 (E)
- net ##454: now also RP8.9 (R8), U53.17 (E)
- net ##432: now reaches U74.21 (VPA)
- net ##432: now also U134.19 (IO1)
- net ##394: now reaches U74.7 (UDS)
- net ##394: now also U126.2 (I2), U130.10 (2D4), U136.2 (I2)
- net ##393: now reaches U74.8 (LDS)
- net ##393: now also U126.3 (I3), U130.9 (2D3), U136.11 (I10)
- net ##431: now reaches U134.2 (I2)
- net ##431: now also U119.13 (IO7), U53.16 (CS_{1})
- net ##450: now reaches U109.4 (A)
- net ##450: now also U110.9 (O0b), U117.13 (A), U133.4 (~{R_{x}C_{B}}), U133.7 (~{TxC_{B}})
- net ##404: now reaches U138.10
- net ##404: now also U53.11 (RS_{1})
- net ##439: now reaches U90.23 (~{CS})
- net ##439: now also U119.16 (IO4)
- net ##449: now reaches U117.10 (A)
- net ##449: now also U110.7 (O1b), U117.4 (A), U133.35 (~{RxC_{A}}), U133.36 (~{TxC_{A}})
- net ##422: now reaches U136.4 (I4)
- net ##422: now also U127.17 (O3)
- net ##430: now reaches U135.5 (Q)
- net ##430: now also U135.12 (D)
- net ##429: now reaches U135.9 (Q)
- net ##429: now also U127.12 (IO8)
- net ##417: now reaches U92.12 (Q4)
- net ##417: now also J?.9 (Pin_9)
- net ##418: now reaches U92.15 (Q5)
- net ##418: now also J?.11 (Pin_11)
- net ##419: now reaches U92.16 (Q6)
- net ##419: now also J?.4 (Pin_4)
- net ##413: now reaches U92.2 (Q0)
- net ##413: now also J?.1 (Pin_1)
- net ##414: now reaches U92.5 (Q1)
- net ##414: now also J?.3 (Pin_3)
- net ##415: now reaches U92.6 (Q2)
- net ##415: now also J?.5 (Pin_5)
- net ##416: now reaches U92.9 (Q3)
- net ##416: now also J?.7 (Pin_7)
- net ##448: now reaches J?.20 (Pin_20)
- net ##448: now also U110.5 (O2b)
- net ##392: now reaches U130.15 (2Q4)
- net ##392: now also U130.6 (1D4)
- net ##390: now reaches U130.16 (2Q3)
- net ##390: now also U130.4 (1D2)
- net ##391: now reaches U130.17 (2Q2)
- net ##391: now also U130.5 (1D3)
- net ##389: now reaches U130.18 (2Q1)
- net ##389: now also U130.3 (1D1)
- net ##396: now reaches U130.19 (1Q4)
- net ##396: now also U127.7 (I7)
- net ##395: now reaches U130.21 (1Q2)
- net ##395: now also U127.6 (I6)
- net ##402: now reaches J1.31 (Pin_31)
- net ##402: now also U138.6
- net ##401: now reaches J1.34 (Pin_34)
- net ##401: now also U138.4
- net ##437: now reaches J1.35 (Pin_35)
- net ##437: now also U126.12 (IO8)
- net ##435: now reaches J1.36 (Pin_36)
- net ##435: now also RP5.5 (R4), U126.5 (I5)
- net ##408: now reaches U137.10
- net ##408: now also U112.14 (O6), U129.10
- net ##405: now reaches U126.19 (IO1)
- net ##405: now also U53.12 (RS_{2})
- net ##403: now reaches U138.8
- net ##403: now also U53.10 (RS_{0})
- net ##407: now reaches U112.15 (O5)
- net ##407: now also U129.9
- net ##442: now reaches U112.9 (I9)
- net ##442: now also U125.15 (TC)
- net ##406: now reaches RP9.2 (R1)
- net ##406: now also U129.1
- net ##440: now reaches U119.14 (IO6)
- net ##440: now also U133.23 (~{CS})
- no-connect marks 31 -> 78
Other:
- moved on the sheet: RP10, RP11, RP4, RP5, RP6, RP7, RP8, RP9

Commit message: rename some nets
Connections:
- net ##1 renamed PROC_D0
- net ##10 renamed PROC_D9
- net ##11 renamed PROC_D10
- net ##12 renamed PROC_D11
- net ##13 renamed PROC_D12
- net ##14 renamed PROC_D13
- net ##15 renamed PROC_D14
- net ##155 renamed ~{PROC_AS}
- net ##156 renamed CLK_32M
- net ##16 renamed PROC_D15
- net ##160 renamed EXT_A19
- net ##177 renamed PROC_R/~{W}
- net ##2 renamed PROC_D1
- net ##220 renamed EXT_A10
- net ##221 renamed EXT_A11
- net ##222 renamed EXT_A12
- net ##223 renamed EXT_A13
- net ##224 renamed EXT_A14
- net ##225 renamed EXT_A15
- net ##226 renamed EXT_A16
- net ##227 renamed EXT_A17
- net ##228 renamed EXT_A18
- net ##230 renamed EXT_A1
- net ##231 renamed EXT_A2
- net ##232 renamed EXT_A3
- net ##233 renamed EXT_A4
- net ##234 renamed EXT_A5
- net ##235 renamed EXT_A6
- net ##236 renamed EXT_A7
- net ##237 renamed EXT_A8
- net ##238 renamed EXT_A9
- net ##240 renamed PROC_A1
- net ##241 renamed PROC_A2
- net ##242 renamed PROC_A3
- net ##243 renamed PROC_A4
- net ##244 renamed PROC_A5
- net ##245 renamed PROC_A6
- net ##246 renamed PROC_A7
- net ##247 renamed PROC_A8
- net ##248 renamed PROC_A9
- net ##249 renamed PROC_A10
- net ##250 renamed PROC_A11
- net ##251 renamed PROC_A12
- net ##252 renamed PROC_A13
- net ##253 renamed PROC_A14
- net ##254 renamed PROC_A15
- net ##255 renamed PROC_A16
- net ##256 renamed PROC_A17
- net ##257 renamed PROC_A18
- net ##258 renamed PROC_A19
- net ##259 renamed PROC_A20
- net ##260 renamed PROC_A21
- net ##261 renamed PROC_A22
- net ##262 renamed PROC_A23
- net ##3 renamed PROC_D2
- net ##337 renamed CLK_8M
- net ##355 renamed EXT_A20
- net ##356 renamed EXT_A21
- net ##357 renamed EXT_A22
- net ##358 renamed EXT_A23
- net ##386 renamed ~{PROC_BERR}
- net ##388 renamed ~{PROC_DTACK}
- net ##393 renamed ~{PROC_LDS}
- net ##394 renamed ~{PROC_UDS}
- net ##398 renamed CLK_4M
- net ##4 renamed PROC_D3
- net ##400 renamed CLK_16M
- net ##5 renamed PROC_D4
- net ##6 renamed PROC_D5
- net ##7 renamed PROC_D6
- net ##8 renamed PROC_D7
- net ##9 renamed PROC_D8
Other:
- moved on the sheet: U138A, U138B, U138C

Commit message: random commit
Connections:
- net ##402 is gone; now on net ~{CLK_8M}: J1.31 (Pin_31), U138.6
- net VCC: now also RP5.1 (common)
- net ##105 renamed ~{BANK_0_CAS}
- net ##106 renamed ~{BANK_1_CAS}
- net ##107 renamed ~{BANK_2_CAS}
- net ##108 renamed ~{BANK_4_CAS}
- net ##109 renamed ~{BANK_3_CAS}
- net ##110 renamed ~{UPPER_DRAM_CAS}
- net ##111 renamed ~{OE_UPPER_ROW_ADDR}
- net ##112 renamed ~{BANK_0_RAS}
- net ##113 renamed ~{BANK_1_RAS}
- net ##114 renamed ~{BANK_2_RAS}
- net ##115 renamed ~{BANK_4_RAS}
- net ##116 renamed ~{BANK_3_RAS}
- net ##117 renamed ~{UPPER_DRAM_RAS}
- net ##126 renamed ~{CLK_32M}
- net ##128 renamed ~{OE_UPPER_COL_ADDR}
- net ##131 renamed PLDWN1
- net ##132 renamed UPPER_~{R}/W
- net ##135: no longer names the net of U105.19 (O1), U113.5 (I5)
- net ##137: no longer names the net of U105.18 (O2), U113.6 (I6)
- net ##138: no longer names the net of U105.17 (O3), U113.7 (I7)
- net ##139: no longer names the net of U105.16 (O4), U113.8 (I8)
- net ##140: no longer names the net of U105.15 (O5), U113.9 (I9)
- net ##141 renamed ~{UPPER_HIGH_PARITY_ERROR}
- net ##142 renamed ~{UPPER_LOW_PARITY_ERROR}
- net ##144: no longer names the net of U105.9 (I9), U128.15 (TC)
- net ##145 renamed PLDWN2
- net ##149 renamed CONSTANT_LOW
- net ##150 renamed ~{ROM_DECODED}
- net ##151 renamed ~{BANK_1_DECODED}
- net ##152 renamed ~{BANK_2_DECODED}
- net ##153 renamed ~{BANK_3_DECODED}
- net ##154 renamed ~{BANK_4_DECODED}
- net ##187 renamed PLUP2
- net ##201 renamed UPPER_DRAM_A0
- net ##202 renamed UPPER_DRAM_A1
- net ##203 renamed UPPER_DRAM_A2
- net ##204 renamed UPPER_DRAM_A3
- net ##205 renamed UPPER_DRAM_A4
- net ##206 renamed UPPER_DRAM_A5
- net ##207 renamed UPPER_DRAM_A6
- net ##208 renamed UPPER_DRAM_A7
- net ##209 renamed UPPER_DRAM_A8
- net ##210 renamed LOWER_DRAM_A0
- net ##211 renamed LOWER_DRAM_A1
- net ##212 renamed LOWER_DRAM_A2
- net ##213 renamed LOWER_DRAM_A3
- net ##214 renamed LOWER_DRAM_A4
- net ##215 renamed LOWER_DRAM_A5
- net ##216 renamed LOWER_DRAM_A6
- net ##217 renamed LOWER_DRAM_A7
- net ##218 renamed LOWER_DRAM_A8
- net ##25 renamed LOWER_DRAM_D0
- net ##26 renamed LOWER_DRAM_D1
- net ##27 renamed LOWER_DRAM_D2
- net ##28 renamed LOWER_DRAM_D3
- net ##29 renamed LOWER_DRAM_D4
- net ##30 renamed LOWER_DRAM_D5
- net ##31 renamed LOWER_DRAM_D6
- net ##317 renamed WRITE_RS232_BAUD
- net ##32 renamed LOWER_DRAM_D7
- net ##325 renamed PLUP1
- net ##33 renamed LOWER_DRAM_D8
- net ##332 renamed ~{CLK_8M}
- net ##333 renamed PLUP3
- net ##338 renamed CLK_1M
- net ##34 renamed LOWER_DRAM_D9
- net ##345 renamed CLK_250K
- net ##35 renamed LOWER_DRAM_D10
- net ##36 renamed LOWER_DRAM_D11
- net ##37 renamed LOWER_DRAM_D12
- net ##38 renamed LOWER_DRAM_D13
- net ##39 renamed LOWER_DRAM_D14
- net ##40 renamed LOWER_DRAM_D15
- net ##401 renamed ~{CLK_16M}
- net ##403 renamed ~{PROC_A1}
- net ##404 renamed ~{PROC_A2}
- net ##411 renamed WRITE_PERIPH_BAUD
- net ##412 renamed WRITE_PANEL
- net ##57 renamed UPPER_DRAM_D8
- net ##58 renamed UPPER_DRAM_D9
- net ##59 renamed UPPER_DRAM_D10
- net ##60 renamed UPPER_DRAM_D11
- net ##61 renamed UPPER_DRAM_D12
- net ##62 renamed UPPER_DRAM_D13
- net ##63 renamed UPPER_DRAM_D14
- net ##64 renamed UPPER_DRAM_D15
- net ##65 renamed UPPER_DRAM_D0
- net ##66 renamed UPPER_DRAM_D1
- net ##67 renamed UPPER_DRAM_D2
- net ##68 renamed UPPER_DRAM_D3
- net ##69 renamed UPPER_DRAM_D4
- net ##70 renamed UPPER_DRAM_D5
- net ##71 renamed UPPER_DRAM_D6
- net ##72 renamed UPPER_DRAM_D7
Other:
- moved on the sheet: J1, J?, RP10, RP11, RP3, RP4, RP5, RP6, RP7, RP8, RP9, U100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
