File: attachment_processor_4/attachment_processor_4.kicad_sch (KiCad schematic)
At the start: 162 parts, among them J1 Conn_02x49_Odd_Even, U1 TMS4256, U10 TMS4256, U100 74ALS576, U101 74ALS842, U102 74ALS841, U103 MC1488, U104 WD1943-PD, U105 TIBPAL16R8, U106 PAL16P8, U107 74ALS576, U108 74ALS841, U109 MC1488, U11 TMS4256, U110 74ALS244, U111 P8274, U112 TIBPAL16R8, U113 TIBPAL16R6, U114 74ALS240, U115 74ALS576, U116 74ALS240, U117 MC1488, U118 74ALS257, U119 PAL16L8, U12 TMS4256, U120 74ALS832, U121 TIBPAL16L8, U122 PAL20L8, U123 CXO_DIP14, U124 MC1489, U125 74ALS161, U126 PAL16R4, U127 TIBPAL16R4, U128 74ALS161, U129 74LS125, U13 TMS4256, U130 74ALS874, U131 74AS576, U132 74ALS257, U133 P8274, U134 PAL16R6, U135 74AS74, U136 PAL16L8, U137 74LS125, U138 74AS1004, U139 74AS161, U14 TMS4256, U140 74AS161, U15 TMS4256, U16 TMS4256, U17 TMS4256, U18 TMS4256, U19 MB81C4256, U2 TMS4256, U20 MB81C4256, U21 MB81C4256, U22 MB81C4256, U23 74F657, U24 74F657, U25 74F657, U26 74F657, U27 TMS4256, U28 TMS4256, U29 TMS4256, U3 TMS4256, U30 TMS4256, U31 TMS4256, U32 TMS4256, U33 TMS4256, U34 TMS4256, U35 TMS4256, U36 TMS4256, U37 TMS4256, U38 TMS4256, U39 TMS4256, U4 TMS4256, U40 TMS4256, U41 TMS4256, U42 TMS4256, U43 TMS4256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

Commit message: Rename some nets
Parts:
- U53: value HD6840 -> HD68B40P
Connections:
- net ##170 renamed PARITY_SELECTION
- net ##192 renamed ~{PROC_IPL2}
- net ##193 renamed ~{PROC_IPL1}
- net ##194 renamed ~{PROC_IPL0}
- net ##343 renamed ~{ACCESSS_FFF00E}
- net ##350 renamed ~{ACCESS_FFF000}
- net ##351 renamed ~{WRITE_FFF004}
- net ##359 renamed ~{ACCESSS_FFF00C}
- net ##361 renamed ~{ACCESSS_FFF00A}
- net ##365 renamed TEST_SW
- net ##368 renamed ~{READ_FFF004}
- net ##387 renamed ~{ACCESS_FFF004}
- net ##431 renamed ~{PTM_CS}
- net ##436 renamed ~{U111_CS}
- net ##439 renamed ~{U90_CS}
- net ##440 renamed ~{U133_CS}
Other:
- note added: "##352 Takes ~D0 when ~{WRITE_FFF004}"
- moved on the sheet: U23, U24, U25, U26, U49, U51, U52, U58, U59, U60, U70, U72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
