File: serial_and_diskette/serial_and_diskette.kicad_sch (KiCad schematic)
At the start: 133 parts, among them U1 74S32, U10 74LS640, U100 74S109, U101 74LS109, U102 Obscured PN, U103 74S109, U104 74S32, U105 74LS74, U106 74LS164, U107 74LS32, U108 74S109, U109 74S08, U11 7438, U110 PAL16P8, U111 74LS04, U113 74S86, U114 WD1935, U115 74LS08, U116 74S08, U117 74LS109, U118 74S32, U119 74S32, U12 74LS74, U120 74LS08, U123 74S00, U124 74LS240, U125 74S04, U126 74S08, U127 74S109, U128 74LS109, U129 74LS74, U13 74LS74, U130 CXO_DIP14_32MHz, U131 HD68B44, U132 74S169, U133 74S74, U134 74LS04, U135 74S11, U136 74S32, U137 74S74, U138 PAL16R8, U139 PAL16R6, U14 74LS08, U140 SN75107B, U142 74S240, U143 A447-0050-02, U144 LM318N, U15 MC14521B, U16 74LS195, U17 Z0801604, U18 74S109, U19 74LS04, U2 74LS09, U20 7438, U21 74LS86, U22 74LS02, U23 74LS02, U24 74LS74, U25 74LS32, U26 74ALS580, U27 74ALS580, U28 3.3k, U29 7438, U3 WD9216, U30 150, U31 74LS14, U32 74LS74, U33 74LS00, U34 74S00, U35 74LS175, U36 74LS04, U37 74ALS580, U38 74LS02, U39 74LS640, U4 74LS161, U40 NE556, U41 74LS08, U42 74LS645, U44 2764, U45 74LS640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

Commit message: Serial/Diskette Adapter: Add Footprints for ICs
Parts:
- U1, U102, U104, U105, U106, U107, U109, U11, U111, U113, U115, U116, U118, U119, U12, U120, U123, U125, U126, U129, U13, U133, U134, U135, U136, U137, U14, U140, U143, U19, U2, U20, U21, U22, U23, U24, U25, U29, U31, U32, U33, U34, U36, U38, U40, U41, U46, U5, U54, U56, U57, U58, U6, U66, U7, U75, U77, U81, U82, U83, U84, U9, U90, U96, U97, U98, U99: footprint (none) -> Package_DIP:DIP-14_W7.62mm
- U10, U110, U124, U138, U139, U142, U26, U27, U37, U39, U42, U45, U47, U48, U51, U52, U53, U61, U62, U64, U67, U69, U72, U74, U85, U87, U89, U92, U93: footprint (none) -> Package_DIP:DIP-20_W7.62mm
- U100, U101, U103, U108, U117, U127, U128, U132, U15, U16, U18, U35, U4, U63, U65, U68, U73, U78, U86, U91: footprint (none) -> Package_DIP:DIP-16_W7.62mm
- U114, U8: footprint (none) -> Package_DIP:DIP-40_W15.24mm
- U144, U3: footprint (none) -> Package_DIP:DIP-8_W7.62mm
- U17: footprint (none) -> Package_DIP:DIP-48_W15.24mm
- U49: footprint (none) -> Package_DIP:DIP-8_W7.62mm_Socket
- U60, U76: footprint (none) -> Package_DIP:DIP-28_W7.62mm
- U71: footprint (none) -> Package_DIP:DIP-64_W22.86mm
